File: template/TXZK-STD-Project/TXZK-STD-Project.kicad_pcb (KiCad board)
At the start: 2 copper layers, 0 parts

Commit message: 添加新的封装并完善工程模板
Other:
- rule pad_to_mask_clearance: 0 -> 0.05
Changed lines of the file:
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@@
 		(35 "F.Fab" user)
 		(33 "B.Fab" user)
-		(39 "User.1" user)
-		(41 "User.2" user)
+		(39 "User.1" user "Fab.VCut")
+		(41 "User.2" user "Fab.EdgeCuts")
 		(43 "User.3" user)
 		(45 "User.4" user)
@@
 	)
 	(setup
-		(pad_to_mask_clearance 0)
+		(stackup
+			(layer "F.SilkS"
+				(type "Top Silk Screen")
+			)
+			(layer "F.Paste"
+				(type "Top Solder Paste")
+			)
+			(layer "F.Mask"
+				(type "Top Solder Mask")
+				(thickness 0.01)
+			)
+			(layer "F.Cu"
+				(type "copper")
+				(thickness 0.035)
+			)
+			(layer "dielectric 1"
+				(type "core")
+				(thickness 1.51)
+				(material "FR4")
+				(epsilon_r 4.5)
+				(loss_tangent 0.02)
+			)
+			(layer "B.Cu"
+				(type "copper")
+				(thickness 0.035)
+			)
+			(layer "B.Mask"
+				(type "Bottom Solder Mask")
+				(thickness 0.01)
+			)
+			(layer "B.Paste"
+				(type "Bottom Solder Paste")
+			)
+			(layer "B.SilkS"
+				(type "Bottom Silk Screen")
+			)
+			(copper_finish "Immersion gold")
+			(dielectric_constraints no)
+		)
+		(pad_to_mask_clearance 0.05)
 		(allow_soldermask_bridges_in_footprints no)
 		(tenting
@@
 	)
 	(embedded_fonts no)
-	(embedded_files
-		(file
-			(name "TXZK-STD-A4-Sheet.kicad_wks")
-			(type worksheet)
-			(data |KLUv/WDQJeUkADZpfSHwGD3QEeyM1dlL9BHR1V16V524kSaE5FqBGWXgGWBgUQF3AHAAcgChlVF+
-				nRwQawzq3O2vHuLW2w4Fu8OWhAsiFm3g7rAW5b0zN8rbPx5Pex69iTa7gz9DdUvGz+Z4Jgx6n6Fa
-				HnHKC/cJ7wIAEBiRNg6lJV2wEei8PQ7efCNB1HlvGoPYUwAEDNfd58uPYPZCjUsFQCAMmTacrfNC
-				hRF1CrcfokR9uZJwMHtQXx5Z6Q3HGPYudJRvOXdFvS75tVZKpc9Z/zXeIO4iquPtkASagMAGc8f6
-				GcM82iesJVzggrhPeHNba/mY1tfdXrRy1NpprXOc9H/M2mutvarWVGKT475Ky637jkEvknCRBweM
-				DEKxVKb12K80E0VFQmGoCNMr/lzsLWHL5bbxiBdGxl74255Wv24MmrSU9WiksNPygFkMQ9xlXfEP
-				dfjz8a/TGTFHcZGDQY8X4oak2L2X0uve+u/0YvP69bdvP0p6zSiveZ0etvYpsYj3trPmXkqv1QMB
-				gz/2199i8qfNk9jlxrs2ySSfaYrGJsNcLo/qbsk0ioiKQH3bmwSzt0ee7kLcsNhzcPU5pV/0Y51+
-				731/vy7Ol7mo8w49h2fpR1ldT3ndWo5NeQ0Qq8G0E8rj8shklr8cF4VDs1AcF0oj2kOrlv/MJIqJ
-				FoFAqOF0Z0ZGkqSQZTdxESGKQMqGdSJQHIMgCIQwFAHLARVDMcgYZoygEGMERAkGWc0ewQjJgeL2
-				w41fz1GDPrFuzXwm8EuRe2WE0qENq8unG69oUHtO88GFMOL6IaAJREAUBDxpIM0PRPnB8uaUDnz6
-				woSb+aGQmxAmg8M2WnWOnryoAKNJA1EORSU5DaoYQ09mepJwemElNJc8IT9sOCg0lPmNScpzLBUU
-				4smETBBL+/WChNHJ56Z8BrWG54cZwshgw4HBe6nBigDJ1BphUeShrWJVJdKGbyOdp/BNO+TECcNC
-				rHdFgkQFBcYpFGzoF5AdpOEWt0OamQbOzqHw2bDIfjyZ3/ypqutzuxc33V7pz/BCs4sWBzZ0r9pR
-				36qDmCESxY52zVnnCW/m/77EONZcNrLbTFUNzFh+8VyMqUDclt8kpX3jnkb7JmgB4z05YX3HBi68
-				oFtxtSAD8SllQomOP1RJLCExx29OvtIjU+lxfcVRRsHyn2heQWWC87lkteBrwWHK3dGXoZH2EHl7
-				LE1IwY602bBiBAlUC6LcsN6mo2IcVwFJv5peOt01BVwSsWDozagTocaZgaDc1ip9yFwI4SdhoRiI
-				BPIV41smd/FGFYlbTiZQAlKEIqoCikRKHjOIJ1OrEjLtuj5mEwfji15gTGeYmNgGXDeuax0lEvRj
-				doB5qRZrF6tdTlHu+ZrscepYc22mWw2S58iCt7wZQPH40eis8EKAKx4tIVAlFEoRiHgSC2rvHzEA
-				qKtQGXP5xVMNsrxSBJSwpR8gDwxeITMphDYrtVW/pAtcq4aqBdsb6KhRG5m4l8hlYrgz65A8tjfb
-				7k/CGqHvECvUO2cfJSPJI7rb1BT4cUp5B/OezxQCprE1yWGrcqQf+aD6tK+u1Bnr6Co=|
-			)
-			(checksum "4B93E79E9BBECA02F2FA9A4A8D9EB107")
-		)
-	)
 )
