File: template/TXZK-STD-Project/TXZK-STD-Project.kicad_sch (KiCad schematic)
At the start: 0 parts

Commit message: 更新部分封装和模板
Other:
- company: (none) -> Company
Changed lines of the file:
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@@
 	(generator_version "10.0")
 	(paper "A3")
+	(title_block
+		(date "Issue Date")
+		(rev "Rev.")
+		(company "Company")
+		(comment 1 "Document No.")
+		(comment 2 "Revision Description")
+		(comment 7 "Previous Rev.")
+		(comment 8 "Previous Issue Date")
+		(comment 9 "Previous Revision Description")
+	)
 	(sheet_instances
 		(path "/"
@@
 		)
 	)
+	(embedded_fonts no)
+	(embedded_files
+		(file
+			(name "TXZK-STD-A3-Sheet.kicad_wks")
+			(type worksheet)
+			(data |KLUv/WBRMM0nAJZuiR7wnDxQGtJA5ZeJ0yLRncw91XKFkJQXW0eJbCJ7UkKIAHYAgABad+2mmjYj
+				jJbbKAqpKtmOwgdd/oiz2HL4inJKHl7GoNwJsshmFC14VgXisshi1c35hlY3t6m04a2EQapPJtmU
+				QTYCPlMebS7LbSmDRPSzsa3LL5sLAEBgxcq2gwjYgo8A37yN7Ce1Ejx8MwhbzpYKgIChdvc79Mfd
+				rcO2VQAEOpTrMwKJNlQhWDZmZOBfuEO8/dHQHa01Zm3GN13Mn4uX1OP0l+2x+ydsD2n9tT6lPqdL
+				2TH2/3THNnNW9GCkLXes0z8gkLlL8sOT/bq7yi+7UbSgBS+/bA5l94opxhNjiXF0/27v7lqhQ0R9
+				7b+6U/fZLbujpn0o5P+tabDdAz7zWBaYyqUhI3xLa9LQ2rKZ2dQheZpGh06byttGusz29LF18Wq1
+				oI8ocY/XdVZ0MaYdJbImf147/tMaFnojy5W2zjpg1GqtMc5apc9/0DtW7WvXdurUH4zzH5xfOx4y
+				7ofasxmULw45hC1lP9iry314EJa6GEVztwRL3RWumOIZAUO75rWdatCfXssTXYf3xvKo+GOzcHwe
+				HI1GIrszD8+CIiPE7gZlEOTullcbFnXWQTUfWdn/sGf0J79rrd7ec45SN/Twzd0W2Wj0B2Xjh7Up
+				orWHc5CYDZ5aLhKNpPPIeD84Z0SziGwyl4gmRspGspGI9n9UFpZN4zG5ZDCPcO1B74F6qJGoNiIj
+				SVLIshvhDSGIOKqmbTIwHAZBEAZhIAKepCGGYxA0BAmKgBgiIIYYItHgAwFVkvSCwyPOvv4kDcJm
+				1lvGJ9x+/+WkjND/UrBC6XSTXAzKE6clubCOlHNDkCBEsASik0oD6Rwiq7BguR+9DiSkE7nN85O6
+				m3xPQ/w2ksCOEF7EFiOTBkouFEWlGn4ehyKfKeI8ebk7moWc15pJgpka6vMNWmloN1pJPAW62VU5
+				JhD6OD37cFNprFqeiR8cKPQCrBRgcP/fNFUEiT/c645diEItZfZMjG+bNeki1TjsxAZGIdgqItH7
+				+mOkYVAgA0xD6sQOpeY0VAqcorIBth3rau5+E18Rt8SmFQ79yaJQF6vgoLOibtqEt1pYOC4hV9Me
+				nLWL8Aa75Aus4wXhyJamo3dgV44A3Q3zAPAPgh4w4D8HK79nhv5RrA+KVXIK6/1wisXAyUrY1omT
+				+LPD1Doh0k2wihsAaKNsDKsEW53WQ7VaOimNA2Z/lnc7xddmXSY4mCLa/7Knj+8I7DFa+Eo9MmIj
+				Cj9+wDpYkVtBQfAmiy8lyIOPFa/p0mYO5ZFmtogJJGHiLulWTP2IuWDqHqNDIoKM3GNyTiS26hPS
+				8FaXmOBOU1iB3XrGxYmFMt8FtmRRU+CLFm6qhJe2Cw9LyAoOiQcOEPuUsJOMxTggygkeYQEJJzjs
+				LDQkEicwdAgHqeTDYTdWfuWBiYz/gPCwnF6QQHFfVnytPC04s49zh4KAI+HceUFNB4PviIzm1Xio
+				0o9PsZDixpwLnZCK565woRwA8pGfqv5RLZ6s/JtDzFTypYiy6hznGmCSWMEX9odmXTiZPtQ1TFF6
+				GaJUdyeBkFRRpNDkEgFdBvY7skVJnKY6U8xeNjZxvLbKKOj6KvxzNQTES+mt1n8iw2anoPHm/8WA
+				U894gy+Mbf7C/DcNgcJiGMOXX7P6C6ZmiBjXwyo=|
+			)
+			(checksum "014D6B121DF5622418FDE556A6DCC1B6")
+		)
+	)

Commit message: 修正模板
Other:
- title: (none) -> Title
Changed lines of the file:
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@@
 	(paper "A3")
 	(title_block
+		(title "Title")
 		(date "Issue Date")
 		(rev "Rev.")
@@
 		(comment 1 "Document No.")
 		(comment 2 "Revision Description")
+		(comment 3 "Revised")
+		(comment 4 "Approved")
+		(comment 5 "Previous Revised")
+		(comment 6 "Previous Approved")
 		(comment 7 "Previous Rev.")
 		(comment 8 "Previous Issue Date")
